File: nrf52832_devboard.kicad_pcb (KiCad board)
At the start: 2 copper layers, 33 x 53.3 mm, 29 parts, among them J1 Conn_01x20_Pin, J2 Conn_01x20_Pin, J3 USB_C_Receptacle_PowerOnly_6P, U1 nRF52832-QFAA, U2 AMS1117-3.3, Y1 32MHz

Commit message: Update BOM
Parts:
- C10: value 12p -> 12p 2%
- C5: value 100p -> 100p NP0 5%
- C7: value 0.8p -> 0.8p NP0 5%
- L1: value 10uH -> 10uH 50mA
- L2: value 15nH -> 15nH RF 10%
- L3: value 3.9nH -> 3.9nH RF 5%
- Y1: value 32MHz -> 32MHz 8pF 40ppm
Changed lines of the file:
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@@
 			)
 		)
-		(property "Value" "0.8p"
+		(property "Value" "0.8p NP0 5%"
 			(at 0 1.16 0)
 			(layer "F.Fab")
@@
 			)
 		)
-		(property "Value" "32MHz"
+		(property "Value" "32MHz 8pF 40ppm"
 			(at 0 2 90)
 			(layer "F.Fab")
@@
 			)
 		)
-		(property "Value" "100p"
+		(property "Value" "100p NP0 5%"
 			(at 0 1.16 90)
 			(layer "F.Fab")
@@
 		(sheetname "Root")
 		(sheetfile "nrf52832_devboard.kicad_sch")
-		(attr exclude_from_pos_files exclude_from_bom)
+		(attr exclude_from_pos_files)
 		(net_tie_pad_groups "1,2")
 		(fp_poly
@@
 			)
 		)
-		(property "Value" "10uH"
+		(property "Value" "10uH 50mA"
 			(at 0 1.43 0)
 			(layer "F.Fab")
@@
 			)
 		)
-		(property "Value" "3.9nH"
+		(property "Value" "3.9nH RF 5%"
 			(at 0 1.17 90)
 			(layer "F.Fab")
@@
 			)
 		)
-		(property "Value" "15nH"
+		(property "Value" "15nH RF 10%"
 			(at 0 1.17 90)
 			(layer "F.Fab")
@@
 			)
 		)
-		(property "Value" "12p"
+		(property "Value" "12p 2%"
 			(at 0 1.16 0)
 			(layer "F.Fab")
@@
 		(sheetname "Root")
 		(sheetfile "nrf52832_devboard.kicad_sch")
-		(attr through_hole exclude_from_bom)
+		(attr through_hole)
 		(fp_poly
 			(pts
