File: nrf52832_devboard.kicad_sch (KiCad schematic)
At the start: 29 parts, among them J1 Conn_01x20_Pin, J2 Conn_01x20_Pin, J3 USB_C_Receptacle_PowerOnly_6P, U1 nRF52832-QFAA, U2 AMS1117-3.3, Y1 32MHz

Commit message: Update BOM
Parts:
- C10: value 12p -> 12p 2%
- C5: value 100p -> 100p NP0 5%
- C7: value 0.8p -> 0.8p NP0 5%
- L1: value 10uH -> 10uH 50mA
- L2: value 15nH -> 15nH RF 10%
- L3: value 3.9nH -> 3.9nH RF 5%
- Y1: value 32MHz -> 32MHz 8pF 40ppm
Changed lines of the file:
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@@
 			)
 		)
-		(property "Value" "32MHz"
-			(at 207.518 105.41 0)
+		(property "Value" "32MHz 8pF 40ppm"
+			(at 201.422 105.156 0)
 			(effects
 				(font
@@
 			)
 		)
-		(property "Value" "12p"
+		(property "Value" "12p 2%"
 			(at 223.52 118.1099 0)
 			(effects
@@
 		(on_board yes)
 		(dnp no)
-		(fields_autoplaced yes)
 		(property "Reference" "L2"
 			(at 207.01 54.61 90)
@@
 			)
 		)
-		(property "Value" "15nH"
-			(at 207.01 57.15 90)
+		(property "Value" "15nH RF 10%"
+			(at 208.28 57.15 90)
 			(effects
 				(font
@@
 			)
 		)
-		(property "Value" "100p"
+		(property "Value" "100p NP0 5%"
 			(at 200.66 39.3699 0)
 			(effects
@@
 			)
 		)
-		(property "Value" "0.8p"
+		(property "Value" "0.8p NP0 5%"
 			(at 194.31 85.0899 0)
 			(effects
@@
 			)
 		)
-		(property "Value" "3.9nH"
+		(property "Value" "3.9nH RF 5%"
 			(at 198.12 76.2 90)
 			(effects
@@
 		(on_board yes)
 		(dnp no)
-		(fields_autoplaced yes)
 		(property "Reference" "L1"
 			(at 194.31 54.61 90)
@@
 			)
 		)
-		(property "Value" "10uH"
-			(at 194.31 57.15 90)
+		(property "Value" "10uH 50mA"
+			(at 193.802 57.15 90)
 			(effects
 				(font
